Commit message: new commit!

File: description/robot.urdf.xacro (robot description, xacro)
@@ -2,3 +2,4 @@
     <robot xmlns:xacro="https://www.ros.org/wiki/xacro" name='robot'>
         <xacro:include filename="robot_core.xacro"/>
+        <xacro:include filename="gazebo_control.xacro"/>
 </robot>

File: description/robot_core.xacro (robot description, xacro)
@@ -35,4 +35,7 @@
         </xacro:inertial_box>
     </link>
+    <gazebo reference="chassis">
+        <material>Gazebo/White</material>
+    </gazebo>
     <link name="left_wheel">
         <visual>
@@ -51,4 +54,7 @@
         </xacro:inertial_cylinder>
     </link>
+    <gazebo reference="left_wheel">
+        <material>Gazebo/Blue</material>
+    </gazebo>
     <link name="right_wheel">
         <visual>
@@ -67,4 +73,7 @@
         </xacro:inertial_cylinder>
     </link>
+    <gazebo reference="right_wheel">
+        <material>Gazebo/Blue</material>
+    </gazebo>
     <link name="caster_wheel">
         <visual>
@@ -83,4 +92,9 @@
         </xacro:inertial_sphere>
     </link>
+    <gazebo reference="caster_wheel">
+        <material>Gazebo/Black</material>
+        <mu1 value="0.001"/>
+        <mu2 value="0.001"/>
+    </gazebo>
 <!--joints!-->
     <joint name="chassis_joint" type="fixed">

Commit message: lidar addition

File: description/robot.urdf.xacro (robot description, xacro)
@@ -3,3 +3,4 @@
         <xacro:include filename="robot_core.xacro"/>
         <xacro:include filename="gazebo_control.xacro"/>
+        <xacro:include filename="lidar.xacro"/>
 </robot>

File: description/robot_core.xacro (robot description, xacro)
@@ -13,4 +13,7 @@
     <material name="black">
         <color rgba="0 0 0 1"/>
+    </material>
+    <material name="red">
+        <color rgba ="1 0 0 1"/>
     </material>
 <!--Links-->
